Commit message: working on 200fps sim not working great.

File: protomotions/data/assets/urdf/for_retargeting/smpl_lower_body.urdf (robot description, URDF)
Before this commit: robot smpl_lower_body, 25 links, 24 joints
Joints:
- joint L_Toe_y: limit lower=-0.35 upper=0 effort=100 velocity=10 -> lower=-0.349066 upper=0.349066 effort=100 velocity=10
- joint R_Toe_y: limit lower=-0.35 upper=0 effort=100 velocity=10 -> lower=-0.349066 upper=0.349066 effort=100 velocity=10
